Commit message: fix(models): restore model-owned placement origins

File: szlab_poly_studio/devices/szlab_mixer_photoshotting/models/device.xacro (robot description, xacro)
@@ -10,5 +10,6 @@
     <link name="${station_name}${device_name}device_link"/>
     <joint name="${station_name}${device_name}device_link_joint" type="fixed">
-      <origin xyz="0 0 0" rpy="0 0 0"/>
+      <!-- Normalize the CAD bbox to the PLR lower-left-bottom origin. -->
+      <origin xyz="0.293683 0.200149 0" rpy="0 0 0"/>
       <parent link="${station_name}${device_name}device_link"/>
       <child link="${station_name}${device_name}base_link"/>

File: szlab_poly_studio/devices/szlab_mixer_pipetting_station/models/device.xacro (robot description, xacro)
@@ -15,5 +15,6 @@
     <link name="${station_name}${device_name}device_link"/>
     <joint name="${station_name}${device_name}device_link_joint" type="fixed">
-      <origin xyz="0 0 0" rpy="0 0 0"/>
+      <!-- Normalize the compound assembly bbox to the PLR lower-left-bottom origin. -->
+      <origin xyz="0.0585 0.033 0" rpy="0 0 0"/>
       <parent link="${station_name}${device_name}device_link"/>
       <child link="${station_name}${device_name}base_link"/>

File: szlab_poly_studio/devices/szlab_mixer_pump/models/device.xacro (robot description, xacro)
@@ -10,5 +10,6 @@
     <link name="${station_name}${device_name}device_link"/>
     <joint name="${station_name}${device_name}device_link_joint" type="fixed">
-      <origin xyz="0 0 0" rpy="0 0 0"/>
+      <!-- Normalize the CAD bbox to the PLR lower-left-bottom origin. -->
+      <origin xyz="0.1425 0.103 0" rpy="0 0 0"/>
       <parent link="${station_name}${device_name}device_link"/>
       <child link="${station_name}${device_name}base_link"/>

File: szlab_poly_studio/devices/szlab_mixer_robot/models/device.xacro (robot description, xacro)
@@ -19,5 +19,6 @@
     <link name="${station_name}${device_name}device_link"/>
     <joint name="${station_name}${device_name}device_link_joint" type="fixed">
-      <origin xyz="0 0 0" rpy="0 0 0"/>
+      <!-- The rail mesh spans y=-0.08..0.08; expose a lower-left base origin. -->
+      <origin xyz="0 0.08 0" rpy="0 0 0"/>
       <parent link="${station_name}${device_name}device_link"/>
       <child link="${station_name}${device_name}arm_slideway"/>

File: szlab_poly_studio/devices/szlab_mixer_stirrer/models/device.xacro (robot description, xacro)
@@ -10,5 +10,6 @@
     <link name="${station_name}${device_name}device_link"/>
     <joint name="${station_name}${device_name}device_link_joint" type="fixed">
-      <origin xyz="0 0 0" rpy="0 0 0"/>
+      <!-- Normalize the CAD bbox to the PLR lower-left-bottom origin. -->
+      <origin xyz="0.355 0.182392 0" rpy="0 0 0"/>
       <parent link="${station_name}${device_name}device_link"/>
       <child link="${station_name}${device_name}base_link"/>

File: szlab_poly_studio/devices/szlab_s07_solid_addition/models/device.xacro (robot description, xacro)
@@ -10,5 +10,6 @@
     <link name="${station_name}${device_name}device_link"/>
     <joint name="${station_name}${device_name}device_link_joint" type="fixed">
-      <origin xyz="0 0 0" rpy="0 0 0"/>
+      <!-- Normalize the CAD bbox to the PLR lower-left-bottom origin. -->
+      <origin xyz="0.38575 0.2515 0" rpy="0 0 0"/>
       <parent link="${station_name}${device_name}device_link"/>
       <child link="${station_name}${device_name}base_link"/>

File: szlab_poly_studio/devices/szlab_s08_cap_station/models/device.xacro (robot description, xacro)
@@ -10,5 +10,6 @@
     <link name="${station_name}${device_name}device_link"/>
     <joint name="${station_name}${device_name}device_link_joint" type="fixed">
-      <origin xyz="0 0 0" rpy="0 0 0"/>
+      <!-- Normalize the compound CAD bbox to the PLR lower-left-bottom origin. -->
+      <origin xyz="0.0545 0.18 0" rpy="0 0 0"/>
       <parent link="${station_name}${device_name}device_link"/>
       <child link="${station_name}${device_name}base_link"/>

File: szlab_poly_studio/resources/szlab_beaker_500ml/models/resource.xacro (robot description, xacro)
@@ -10,5 +10,6 @@
     <link name="${station_name}${device_name}device_link"/>
     <joint name="${station_name}${device_name}device_link_joint" type="fixed">
-      <origin xyz="0 0 0" rpy="0 0 0"/>
+      <!-- PLR stores the container lower-left; put the vessel axis at the site center. -->
+      <origin xyz="0.043 0.043 0" rpy="0 0 0"/>
       <parent link="${station_name}${device_name}device_link"/>
       <child link="${station_name}${device_name}base_link"/>

File: szlab_poly_studio/resources/szlab_liquid_reagent_bottle_100ml/models/resource.xacro (robot description, xacro)
@@ -10,5 +10,6 @@
     <link name="${station_name}${device_name}device_link"/>
     <joint name="${station_name}${device_name}device_link_joint" type="fixed">
-      <origin xyz="0 0 0" rpy="0 0 0"/>
+      <!-- PLR stores the container lower-left; put the bottle axis at the site center. -->
+      <origin xyz="0.028 0.028 0" rpy="0 0 0"/>
       <parent link="${station_name}${device_name}device_link"/>
       <child link="${station_name}${device_name}base_link"/>

File: szlab_poly_studio/resources/szlab_poly_beaker_warehouse/models/resource.xacro (robot description, xacro)
@@ -10,5 +10,6 @@
     <link name="${station_name}${device_name}device_link"/>
     <joint name="${station_name}${device_name}device_link_joint" type="fixed">
-      <origin xyz="0 0 0" rpy="0 0 0"/>
+      <!-- Normalize the carrier CAD bbox to its PLR lower-left-bottom origin. -->
+      <origin xyz="0.394994 0.1 0" rpy="0 0 0"/>
       <parent link="${station_name}${device_name}device_link"/>
       <child link="${station_name}${device_name}base_link"/>

File: szlab_poly_studio/resources/szlab_poly_powder_container_placeholder_warehouse/models/resource.xacro (robot description, xacro)
@@ -10,5 +10,6 @@
     <link name="${station_name}${device_name}device_link"/>
     <joint name="${station_name}${device_name}device_link_joint" type="fixed">
-      <origin xyz="0 0 0" rpy="0 0 0"/>
+      <!-- Turn the CAD into deck orientation, then normalize its rotated bbox. -->
+      <origin xyz="0.184986 0.05 0" rpy="0 0 1.5707963267948966"/>
       <parent link="${station_name}${device_name}device_link"/>
       <child link="${station_name}${device_name}base_link"/>

File: szlab_poly_studio/resources/szlab_poly_s10_liquid_reagent_placeholder_warehouse/models/resource.xacro (robot description, xacro)
@@ -10,5 +10,6 @@
     <link name="${station_name}${device_name}device_link"/>
     <joint name="${station_name}${device_name}device_link_joint" type="fixed">
-      <origin xyz="0 0 0" rpy="0 0 0"/>
+      <!-- Normalize the carrier CAD bbox to its PLR lower-left-bottom origin. -->
+      <origin xyz="0.279986 0.06 0" rpy="0 0 0"/>
       <parent link="${station_name}${device_name}device_link"/>
       <child link="${station_name}${device_name}base_link"/>

File: szlab_poly_studio/resources/szlab_poly_s1_loading_buffer_warehouse/models/resource.xacro (robot description, xacro)
@@ -10,5 +10,6 @@
     <link name="${station_name}${device_name}device_link"/>
     <joint name="${station_name}${device_name}device_link_joint" type="fixed">
-      <origin xyz="0 0 0" rpy="0 0 0"/>
+      <!-- Turn the CAD into deck orientation, then normalize its rotated bbox. -->
+      <origin xyz="0.23492 0.135083 0" rpy="0 0 1.5707963267948966"/>
       <parent link="${station_name}${device_name}device_link"/>
       <child link="${station_name}${device_name}base_link"/>

File: szlab_poly_studio/resources/szlab_poly_s2_tip_placeholder_warehouse/models/resource.xacro (robot description, xacro)
@@ -10,5 +10,6 @@
     <link name="${station_name}${device_name}device_link"/>
     <joint name="${station_name}${device_name}device_link_joint" type="fixed">
-      <origin xyz="0 0 0" rpy="0 0 0"/>
+      <!-- Normalize the carrier CAD bbox to its PLR lower-left-bottom origin. -->
+      <origin xyz="0.155012 0.07 0" rpy="0 0 0"/>
       <parent link="${station_name}${device_name}device_link"/>
       <child link="${station_name}${device_name}base_link"/>

File: szlab_poly_studio/resources/szlab_powder_container/models/resource.xacro (robot description, xacro)
@@ -10,5 +10,6 @@
     <link name="${station_name}${device_name}device_link"/>
     <joint name="${station_name}${device_name}device_link_joint" type="fixed">
-      <origin xyz="0 0 0" rpy="0 0 0"/>
+      <!-- PLR stores the container lower-left; put the vessel axis at the site center. -->
+      <origin xyz="0.035 0.035 0" rpy="0 0 0"/>
       <parent link="${station_name}${device_name}device_link"/>
       <child link="${station_name}${device_name}base_link"/>

File: szlab_poly_studio/resources/szlab_sample_vial_500ml/models/resource.xacro (robot description, xacro)
@@ -10,5 +10,6 @@
     <link name="${station_name}${device_name}device_link"/>
     <joint name="${station_name}${device_name}device_link_joint" type="fixed">
-      <origin xyz="0 0 0" rpy="0 0 0"/>
+      <!-- PLR stores the container lower-left; put the vessel axis at the site center. -->
+      <origin xyz="0.043 0.043 0" rpy="0 0 0"/>
       <parent link="${station_name}${device_name}device_link"/>
       <child link="${station_name}${device_name}base_link"/>

File: szlab_poly_studio/resources/szlab_tip_box/models/resource.xacro (robot description, xacro)
@@ -10,5 +10,6 @@
     <link name="${station_name}${device_name}device_link"/>
     <joint name="${station_name}${device_name}device_link_joint" type="fixed">
-      <origin xyz="0 0 0" rpy="0 0 0"/>
+      <!-- Normalize the tip-box CAD bbox to the PLR lower-left-bottom origin. -->
+      <origin xyz="0.043 0.06403 0" rpy="0 0 0"/>
       <parent link="${station_name}${device_name}device_link"/>
       <child link="${station_name}${device_name}base_link"/>
