Commit message: fix(models): align pre-oriented warehouse meshes

File: szlab_poly_studio/resources/szlab_poly_powder_container_placeholder_warehouse/models/resource.xacro (robot description, xacro)
@@ -10,6 +10,6 @@
     <link name="${station_name}${device_name}device_link"/>
     <joint name="${station_name}${device_name}device_link_joint" type="fixed">
-      <!-- Turn the CAD into deck orientation, then normalize its rotated bbox. -->
-      <origin xyz="0.184986 0.05 0" rpy="0 0 1.5707963267948966"/>
+      <!-- The latest STL is pre-oriented; normalize its bbox to the PLR origin. -->
+      <origin xyz="0.05 0.185014 0" rpy="0 0 0"/>
       <parent link="${station_name}${device_name}device_link"/>
       <child link="${station_name}${device_name}base_link"/>

File: szlab_poly_studio/resources/szlab_poly_s1_loading_buffer_warehouse/models/resource.xacro (robot description, xacro)
@@ -10,6 +10,6 @@
     <link name="${station_name}${device_name}device_link"/>
     <joint name="${station_name}${device_name}device_link_joint" type="fixed">
-      <!-- Turn the CAD into deck orientation, then normalize its rotated bbox. -->
-      <origin xyz="0.23492 0.135083 0" rpy="0 0 1.5707963267948966"/>
+      <!-- The latest STL is pre-oriented; center it on the 200 x 442 mm footprint. -->
+      <origin xyz="0.100083 0.22108 0" rpy="0 0 0"/>
       <parent link="${station_name}${device_name}device_link"/>
       <child link="${station_name}${device_name}base_link"/>
