Commit message: 更新机械臂模型

File: szlab_poly_studio/devices/szlab_mixer_robot/models/config/macro.ros2_control.xacro (robot description, xacro)
@@ -14,43 +14,43 @@
                 <state_interface name="velocity"/>
             </joint>
-            <joint name="${device_name}eco65_joint_1">
+            <joint name="${device_name}cr7_joint_1">
                 <command_interface name="position"/>
                 <state_interface name="position">
-                  <param name="initial_value">${initial_positions['eco65_joint_1']}</param>
+                  <param name="initial_value">${initial_positions['cr7_joint_1']}</param>
                 </state_interface>
                 <state_interface name="velocity"/>
             </joint>
-            <joint name="${device_name}eco65_joint_2">
+            <joint name="${device_name}cr7_joint_2">
                 <command_interface name="position"/>
                 <state_interface name="position">
-                  <param name="initial_value">${initial_positions['eco65_joint_2']}</param>
+                  <param name="initial_value">${initial_positions['cr7_joint_2']}</param>
                 </state_interface>
                 <state_interface name="velocity"/>
             </joint>
-            <joint name="${device_name}eco65_joint_3">
+            <joint name="${device_name}cr7_joint_3">
                 <command_interface name="position"/>
                 <state_interface name="position">
-                  <param name="initial_value">${initial_positions['eco65_joint_3']}</param>
+                  <param name="initial_value">${initial_positions['cr7_joint_3']}</param>
                 </state_interface>
                 <state_interface name="velocity"/>
             </joint>
-            <joint name="${device_name}eco65_joint_4">
+            <joint name="${device_name}cr7_joint_4">
                 <command_interface name="position"/>
                 <state_interface name="position">
-                  <param name="initial_value">${initial_positions['eco65_joint_4']}</param>
+                  <param name="initial_value">${initial_positions['cr7_joint_4']}</param>
                 </state_interface>
                 <state_interface name="velocity"/>
             </joint>
-            <joint name="${device_name}eco65_joint_5">
+            <joint name="${device_name}cr7_joint_5">
                 <command_interface name="position"/>
                 <state_interface name="position">
-                  <param name="initial_value">${initial_positions['eco65_joint_5']}</param>
+                  <param name="initial_value">${initial_positions['cr7_joint_5']}</param>
                 </state_interface>
                 <state_interface name="velocity"/>
             </joint>
-            <joint name="${device_name}eco65_joint_6">
+            <joint name="${device_name}cr7_joint_6">
                 <command_interface name="position"/>
                 <state_interface name="position">
-                  <param name="initial_value">${initial_positions['eco65_joint_6']}</param>
+                  <param name="initial_value">${initial_positions['cr7_joint_6']}</param>
                 </state_interface>
                 <state_interface name="velocity"/>

File: szlab_poly_studio/devices/szlab_mixer_robot/models/config/macro.srdf.xacro (robot description, xacro)
@@ -3,14 +3,18 @@
     <xacro:macro name="szlab_mixer_robot_srdf" params="device_name">
         <group name="${device_name}arm">
-            <chain base_link="${device_name}arm_slideway" tip_link="${device_name}eco65_link_6"/>
+            <chain base_link="${device_name}arm_slideway" tip_link="${device_name}cr7_link_6"/>
         </group>
-        <disable_collisions link1="${device_name}arm_slideway" link2="${device_name}eco65_base" reason="Adjacent"/>
-        <disable_collisions link1="${device_name}eco65_base" link2="${device_name}eco65_link_1" reason="Adjacent"/>
-        <disable_collisions link1="${device_name}eco65_link_1" link2="${device_name}eco65_link_2" reason="Adjacent"/>
-        <disable_collisions link1="${device_name}eco65_link_2" link2="${device_name}eco65_link_3" reason="Adjacent"/>
-        <disable_collisions link1="${device_name}eco65_link_3" link2="${device_name}eco65_link_4" reason="Adjacent"/>
-        <disable_collisions link1="${device_name}eco65_link_4" link2="${device_name}eco65_link_5" reason="Adjacent"/>
-        <disable_collisions link1="${device_name}eco65_link_5" link2="${device_name}eco65_link_6" reason="Adjacent"/>
-        <disable_collisions link1="${device_name}arm_slideway" link2="${device_name}eco65_link_1" reason="Never"/>
+        <disable_collisions link1="${device_name}arm_slideway" link2="${device_name}cr7_base" reason="Adjacent"/>
+        <disable_collisions link1="${device_name}arm_slideway" link2="${device_name}cr7_link_1" reason="Never"/>
+        <disable_collisions link1="${device_name}cr7_base" link2="${device_name}cr7_link_1" reason="Adjacent"/>
+        <disable_collisions link1="${device_name}cr7_base" link2="${device_name}cr7_link_2" reason="Never"/>
+        <disable_collisions link1="${device_name}cr7_base" link2="${device_name}cr7_link_4" reason="Never"/>
+        <disable_collisions link1="${device_name}cr7_link_1" link2="${device_name}cr7_link_2" reason="Adjacent"/>
+        <disable_collisions link1="${device_name}cr7_link_1" link2="${device_name}cr7_link_4" reason="Never"/>
+        <disable_collisions link1="${device_name}cr7_link_2" link2="${device_name}cr7_link_3" reason="Adjacent"/>
+        <disable_collisions link1="${device_name}cr7_link_3" link2="${device_name}cr7_link_4" reason="Adjacent"/>
+        <disable_collisions link1="${device_name}cr7_link_4" link2="${device_name}cr7_link_5" reason="Adjacent"/>
+        <disable_collisions link1="${device_name}cr7_link_4" link2="${device_name}cr7_link_6" reason="Never"/>
+        <disable_collisions link1="${device_name}cr7_link_5" link2="${device_name}cr7_link_6" reason="Adjacent"/>
     </xacro:macro>
 </robot>
