Commit message: 添加移液站位置，将整个磁搅模块拆成6个单独模块

File: szlab_poly_studio/devices/szlab_mixer_pipetting_station/models/device.xacro (robot description, xacro)
@@ -15,6 +15,6 @@
     <link name="${station_name}${device_name}device_link"/>
     <joint name="${station_name}${device_name}device_link_joint" type="fixed">
-      <!-- Normalize the compound assembly bbox to the PLR lower-left-bottom origin. -->
-      <origin xyz="0.0585 0.033 0" rpy="0 0 0"/>
+      <!-- 原点=底板左下角底面，与 shape.yml / PLR seat 同一坐标系；勿再加 bbox 平移。 -->
+      <origin xyz="0 0 0" rpy="0 0 0"/>
       <parent link="${station_name}${device_name}device_link"/>
       <child link="${station_name}${device_name}base_link"/>
@@ -44,7 +44,7 @@
       </collision>
     </link>
-    <!-- 2) 原移液枪模组底座：左下角 → 底板 (4, 388, 12) mm -->
+    <!-- 2) 原移液枪模组底座：左下角 → 底板 (4, 388, 12) mm；joint = target - mesh_aabb_min -->
     <joint name="${station_name}${device_name}pipetting_station_joint" type="fixed">
-      <origin xyz="0.2615 0.429 0.012" rpy="0 0 0"/>
+      <origin xyz="0.324 0.429 0.012" rpy="0 0 0"/>
       <parent link="${station_name}${device_name}base_link"/>
       <child link="${station_name}${device_name}pipetting_station"/>

File: szlab_poly_studio/devices/szlab_mixer_stirrer/models/device.xacro (robot description, xacro)
@@ -1,4 +1,9 @@
 <?xml version="1.0" encoding="utf-8"?>
 <robot xmlns:xacro="http://www.ros.org/wiki/xacro">
+  <!-- Individual S04 magnetic-stirrer module (单独磁搅模块).
+       CAD hot-plate (the model center) sits at (-0.225, +0.050) — i.e. +50 mm in Y from
+       the rack bottom center, which shares the same CAD origin as the rack.
+       device_link uses PLR lower-left-bottom; the plate lands at (0.108914, 0.226618,
+       0.122121) in device_link, and the beaker seat sits on it. -->
   <xacro:macro name="szlab_mixer_stirrer" params="parent_link:='' station_name:='' device_name:='' x:=0 y:=0 z:=0 rx:=0 ry:=0 r:=0 mesh_path:=''">
     <joint name="${station_name}${device_name}base_link_joint" type="fixed">
@@ -10,6 +15,6 @@
     <link name="${station_name}${device_name}device_link"/>
     <joint name="${station_name}${device_name}device_link_joint" type="fixed">
-      <!-- Normalize the CAD bbox to the PLR lower-left-bottom origin. -->
-      <origin xyz="0.355 0.182392 0" rpy="0 0 0"/>
+      <!-- PLR lower-left-bottom of the CAD bbox. -->
+      <origin xyz="0.33391374 0.17660786 -0.008" rpy="0 0 0"/>
       <parent link="${station_name}${device_name}device_link"/>
       <child link="${station_name}${device_name}base_link"/>
@@ -18,7 +23,7 @@
     <link name="${station_name}${device_name}base_link">
       <inertial>
-        <origin xyz="0.00090138410687518 5.94790366356263E-05 0.376988397961134" rpy="0 0 0"/>
-        <mass value="45.5919699023364"/>
-        <inertia ixx="1.10758909875164" ixy="-8.76425304011537E-06" ixz="1.58242458961115E-05" iyy="1.88685362178322" iyz="-1.67297882958595E-06" izz="1.59431437186427"/>
+        <origin xyz="-0.225338277133257 -0.00110785614684515 0.0139081948746832" rpy="0 0 0"/>
+        <mass value="0.0808795174685058"/>
+        <inertia ixx="1.01374773273621E-05" ixy="-3.78864870740827E-22" ixz="1.53792985157028E-21" iyy="1.01374773273621E-05" iyz="5.86569718155341E-21" izz="1.80459170576023E-05"/>
       </inertial>
       <visual>
@@ -28,5 +33,5 @@
         </geometry>
         <material name="">
-          <color rgba="0.752941176470588 0.752941176470588 0.752941176470588 1"/>
+          <color rgba="0.698039215686274 0.698039215686274 0.698039215686274 1"/>
         </material>
       </visual>
